Commit message: Add gravity-compensated sliding effort controller with matched-PD validation

File: simulation/meituan_sim/urdf/aubo_S3_gazebo.urdf.xacro (robot description, xacro)
@@ -28,4 +28,6 @@
     <xacro:hook parent="flange"/>
   </xacro:if>
+  <xacro:arg name="command_interface" default="position"/>
+  <xacro:property name="control_interface" value="$(arg command_interface)"/>
   <ros2_control name="aubo_S3_gazebo" type="system">
     <hardware>
@@ -37,7 +39,9 @@
     <xacro:macro name="s3_joint" params="name init">
       <joint name="${name}">
-        <command_interface name="position">
+        <command_interface name="${control_interface}">
+          <xacro:if value="${control_interface == 'position'}">
           <param name="min">${-2*pi}</param>
           <param name="max">${2*pi}</param>
+          </xacro:if>
         </command_interface>
         <state_interface name="position"><param name="initial_value">${init}</param></state_interface>
